Commit message: tut krok 12.1

File: description/colors.xacro (robot description, xacro)
@@ -13,3 +13,6 @@
     <color rgba="0 0 0 1"/>
 </material>
+<material name="red">
+    <color rgba="1 0 0 1"/>
+</material>
 </robot>

File: description/robot.urdf.xacro (robot description, xacro)
@@ -4,5 +4,8 @@
   <xacro:include filename="colors.xacro"/>
   <xacro:include filename="robot_core.xacro"/>
-  <xacro:include filename="gazebo_control.xacro"/>
+ <!-- <xacro:include filename="gazebo_control.xacro"/> -->
+  <xacro:include filename="ros2_control.xacro" />
+  <xacro:include filename="lidar.xacro"/>
+  <xacro:include filename="camera.xacro" />
 <!-- <link name="base_link">  </link> -->
 </robot>
